File: Hardware2/Board/LedControl.sch (KiCad schematic (older format))
At the start: 27 parts

Commit message: Finished schematic
Parts:
- removed P? (x2): CONN_01X04, symbol CONN_01X04
- removed P?: CONN_01X07, symbol CONN_01X07
- removed R? (x2): 10k, symbol R
- added J1: CONN_01X02, LedControl:Jumper, symbol CONN_01X02
- added J2: CONN_01X03, LedControl:Jumper3, symbol CONN_01X03
- added P10, P12, P13, P14, P2, P3, P4, P5, P6, P7, P8, P9: CONN_01X01, LedControl:Pad, symbol CONN_01X01
- added P17, P18: CONN_01X02, LedControl:WAGO_2059-302, symbol CONN_01X02
- added R4: 100k, Resistors_SMD:R_0603, symbol R
- added U2: SP3078, Housings_SOIC:SOIC-8_3.9x4.9mm_Pitch1.27mm, symbol SP3485CN
- C1, C2, C3, C4: renamed from C?; footprint (none) -> Capacitors_SMD:C_0603
- C5: renamed from C?; value 4u7 -> 10u; footprint (none) -> Capacitors_SMD:C_1206
- D1: renamed from D?; footprint (none) -> LEDs:LED_0805
- P1: renamed from P?; footprint (none) -> Connect:USB_Mini-B
- P11: renamed from U?; footprint (none) -> LedControl:MicroSD
- P15, P20: renamed from P?; footprint (none) -> Pin_Headers:Pin_Header_Straight_1x03
- P16: renamed from P?; footprint (none) -> LedControl:Connector_Flat_24_Pitch0.50mm
- P19: renamed from P?; footprint (none) -> LedControl:WAGO_2059-302
- R1, R2: renamed from R?; footprint (none) -> Resistors_SMD:R_0603
- R3: renamed from R?; value 900k -> 1M2; footprint (none) -> Resistors_SMD:R_0603
- R5: renamed from R?; value 10k -> 100k; footprint (none) -> Resistors_SMD:R_0603
- SW1, SW2: renamed from SW?; footprint (none) -> LedControl:ALPS_BOURNS_EC12
- U1: renamed from U?; footprint LQFP48 -> Housings_QFP:LQFP-48_7x7mm_Pitch0.5mm
- U3: renamed from U?; footprint SO-8 -> Housings_SOIC:SOIC-8_3.9x4.9mm_Pitch1.27mm
- X1: renamed from X?; footprint (none) -> LedControl:CSTCE_16
- X2: renamed from X?; footprint (none) -> LedControl:Oscillator_5x3.2mm
Connections:
- net labels added: VCC
- net labels removed: +12V
- wire segments 191 -> 177
Other:
- note added: "DISPLAY\nSSD1309"
- note added: "GND"
- note added: "R = (Vcc - 3.3V) / 10uA"
- note added: "RS485"
- note added: "RS485_DE"
- note added: "RS485_RX"
- note added: "RS485_TX"
- note added: "SD_Cd"
- note removed: "DISPLAY"
- note removed: "EN12V"

Commit message: Finished routing main board
Parts:
- removed P10, P12, P9: CONN_01X01, LedControl:Pad, symbol CONN_01X01
- removed U1: STM32L151CCTx, Housings_QFP:LQFP-48_7x7mm_Pitch0.5mm, symbol STM32L151CCTx
- removed X1: CRYSTAL_SMD, LedControl:CSTCE_16, symbol CRYSTAL_SMD
- added J3: CONN_01X02, LedControl:Jumper, symbol CONN_01X02
- added P11: 2059-302, LedControl:WAGO_2059-302, symbol CONN_01X02
- added P14: TP, LedControl:Pad, symbol CONN_01X01
- added R10, R2, R4, R6, R9: 120R, Resistors_SMD:R_1206, symbol R
- added R3: 523k, Resistors_SMD:R_0603, symbol R
- added U1: STM32L433CCUx, Housings_DFN_QFN:QFN-48-1EP_7x7mm_Pitch0.5mm, symbol STM32L433CCUx
- added U2: SP485CN, Housings_SOIC:SOIC-8_3.9x4.9mm_Pitch1.27mm, symbol SP3485CN
- J1: value CONN_01X02 -> J
- J2: value CONN_01X03 -> J
- P1: footprint Connect:USB_Mini-B -> LedControl:Micro_USB
- P10: renamed from P8; value CONN_01X01 -> TP
- P12: renamed from P16; value CONN_01X24 -> DISPLAY
- P13: renamed from P14; value CONN_01X01 -> TP
- P16: renamed from P17; value CONN_01X02 -> 2059-302
- P17: renamed from P19; value CONN_01X02 -> 2059-302
- P2: renamed from P13; value CONN_01X01 -> TP
- P3: renamed from P2; value CONN_01X01 -> TP
- P4: renamed from P3; value CONN_01X01 -> TP
- P5: renamed from P18; value CONN_01X02 -> 2059-302
- P6: renamed from P4; value CONN_01X01 -> TP
- P7: renamed from P5; value CONN_01X01 -> TP
- P8: renamed from P11; footprint LedControl:MicroSD -> LedControl:Micro_SD
- P9: renamed from P7; value CONN_01X01 -> TP
- R5: renamed from R3; value 1M2 -> 523k
- R8: renamed from R2; value 470R -> 120R; footprint Resistors_SMD:R_0603 -> Resistors_SMD:R_1206
- SW1, SW2: value ROTARY_ENCODER_SWITCH -> PEC12R-4215F-S0024
- U3: renamed from U2; value SP3078 -> SP485CN
- renumbered P6 to P15, P20 to P18, P15 to P19, R5 to R11, R4 to R7, U3 to U4, X2 to X1
Connections:
- wire segments 177 -> 199
Other:
- note added: "DISPLAY\nSSD1309\nSPI2"
- note added: "ENCODER 1\nTIM1"
- note added: "ENCODER 2\nTIM2"
- note added: "LED STRIP\nUSART1"
- note added: "RS485\nGND/PWR"
- note added: "RS485\nUSART2"
- note added: "RS485\nUSART3"
- note added: "SD CARD\nSPI1"
- note added: "SPI1_SD_MISO"
- note added: "SPI1_SD_MOSI"
- note added: "SPI1_SD_NSS"
- note added: "SPI1_SD_SCK"
- note added: "SPI2_DISP_MOSI"
- note added: "SPI2_DISP_NSS"
- note added: "SPI2_DISP_SCK"
- note added: "TIM1_ENC1_CH1"
- note added: "TIM1_ENC1_CH2"
- note added: "TIM2_ENC2_CH1"
- note added: "TIM2_ENC2_CH2"
- note added: "USART1"
- note added: "USART1_LED_TX"
- note added: "USART1_RX"
- note added: "USART2_RS485_DE"
- note added: "USART2_RS485_RX"
- note added: "USART2_RS485_TX"
- note added: "USART3_RS485_DE"
- note added: "USART3_RS485_RX"
- note added: "USART3_RS485_TX"
- note removed: "BOOT_LED_TX"
- note removed: "BOOT_RX"
- note removed: "DISPLAY\nSSD1309"
- note removed: "DISP_CS#"
- note removed: "DISP_MOSI"
- note removed: "DISP_SCK"
- note removed: "ENC1_A"
- note removed: "ENC1_B"
- note removed: "ENC2_A"
- note removed: "ENC2_B"
- note removed: "LED STRIP"
- note removed: "RS485"
- note removed: "RS485_DE"
- note removed: "RS485_RX"
- note removed: "RS485_TX"
- note removed: "SD CARD"
- note removed: "SD_MISO"
- note removed: "SD_MOSI"
- note removed: "SD_SCK"
- note removed: "SD_SS"
- note removed: "SPI1_MISO"
- note removed: "SPI1_MOSI"
- note removed: "SPI1_SCK"
- moved on the sheet: U3

Commit message: routing nearly finished
Parts:
- removed R5: 523k, Resistors_SMD:R_0603, symbol R
- added P32, P33: TP, LedControl:Pad, symbol CONN_01X01
- R11: value 100k -> 10k
- R3: value 523k -> 1M2
- R7: value 100k -> 52k3
Connections:
- wire segments 199 -> 211
Other:
- note added: "ADC1_IN12_U1"
- note added: "ADC1_IN15_U2"
- note added: "D0/SCK"
- note added: "D1/MOSI"
- note added: "LED1\nUSART1"
- note added: "LED2\nUSART2"
- note added: "LED2_DE"
- note added: "USART1_LED1_TX"
- note added: "USART2_LED2_RX"
- note added: "USART2_LED2_TX"
- note removed: "D0 (SCK)"
- note removed: "D1 (MOSI)"
- note removed: "LED STRIP\nUSART1"
- note removed: "RS485\nUSART2"
- note removed: "USART1_LED_TX"
- note removed: "USART2_RS485_DE"
- note removed: "USART2_RS485_RX"
- note removed: "USART2_RS485_TX"

Commit message: Start software for stm32 based hardware2
Other:
- note added: "ENC1_TIM1_CH1"
- note added: "ENC1_TIM1_CH2"
- note added: "ENC2_TIM2_CH1"
- note added: "ENC2_TIM2_CH2"
- note added: "RS485_USART3_DE"
- note added: "RS485_USART3_RX"
- note added: "RS485_USART3_TX"
- note added: "SD_SPI1_MISO"
- note added: "SD_SPI1_MOSI"
- note added: "SD_SPI1_SCK"
- note added: "STRIP1\nUSART1"
- note added: "STRIP1_USART1_TX"
- note added: "STRIP2\nUSART2"
- note added: "STRIP2_DE"
- note added: "STRIP2_USART2_RX"
- note added: "STRIP2_USART2_TX"
- note added: "U1_ADC1_IN12"
- note added: "U2_ADC1_IN15"
- note removed: "ADC1_IN12_U1"
- note removed: "ADC1_IN15_U2"
- note removed: "LED1\nUSART1"
- note removed: "LED2\nUSART2"
- note removed: "LED2_DE"
- note removed: "SPI1_SD_MISO"
- note removed: "SPI1_SD_MOSI"
- note removed: "SPI1_SD_SCK"
- note removed: "TIM1_ENC1_CH1"
- note removed: "TIM1_ENC1_CH2"
- note removed: "TIM2_ENC2_CH1"
- note removed: "TIM2_ENC2_CH2"
- note removed: "USART1_LED1_TX"
- note removed: "USART2_LED2_RX"
- note removed: "USART2_LED2_TX"
- note removed: "USART3_RS485_DE"
- note removed: "USART3_RS485_RX"
- note removed: "USART3_RS485_TX"
Changed lines of the file:
@@
 $EndComp
 Text Notes 10400 5350 0    60   ~ 0
-LED1\nUSART1
+STRIP1\nUSART1
 Text Notes 1700 5600 0    60   ~ 0
 DISPLAY\nSSD1309\nSPI2
@@
 ENC2_SW
 Text Notes 5550 2950 0    60   ~ 0
-TIM1_ENC1_CH1
+ENC1_TIM1_CH1
 Text Notes 5550 3050 0    60   ~ 0
-TIM1_ENC1_CH2
+ENC1_TIM1_CH2
 Text Notes 4550 1950 0    60   ~ 0
 ENC1_SW
@@
 SPI2_DISP_MOSI
 Text Notes 4550 2850 0    60   ~ 0
-USART1_LED1_TX
+STRIP1_USART1_TX
 Text Notes 4550 3150 0    60   ~ 0
 DEBUG_LED
@@
 DISP_RES#
 Text Notes 4550 2750 0    60   ~ 0
-SPI1_SD_MOSI
+SD_SPI1_MOSI
 Text Notes 5700 2650 0    60   ~ 0
-SPI1_SD_SCK
+SD_SPI1_SCK
 Text Notes 5550 2250 0    60   ~ 0
-TIM2_ENC2_CH2
+ENC2_TIM2_CH2
 Text Notes 5550 2150 0    60   ~ 0
-TIM2_ENC2_CH1
+ENC2_TIM2_CH1
 $Comp
 L +3.3V #PWR011
@@
 $EndComp
 Text Notes 5650 2750 0    60   ~ 0
-SPI1_SD_MISO
+SD_SPI1_MISO
 $Comp
 L VCC #PWR019
@@
 Connection ~ 6000 5500
 Text Notes 4600 3250 0    60   ~ 0
-USART3_RS485_TX
+RS485_USART3_TX
 Text Notes 4600 3350 0    60   ~ 0
-USART3_RS485_RX
+RS485_USART3_RX
 Text Notes 4550 2350 0    60   ~ 0
-USART3_RS485_DE
+RS485_USART3_DE
 $Comp
 L SP3485CN U3
@@
 USART1
 Text Notes 4550 1850 0    60   ~ 0
-LED2_DE
-Text Notes 5500 2350 0    60   ~ 0
-USART2_LED2_TX
-Text Notes 5500 2450 0    60   ~ 0
-USART2_LED2_RX
+STRIP2_DE
+Text Notes 5450 2350 0    60   ~ 0
+STRIP2_USART2_TX
+Text Notes 5450 2450 0    60   ~ 0
+STRIP2_USART2_RX
 Wire Wire Line
 	8100 2700 8500 2700
@@
 	950  2000 950  1900
 Text Notes 650  4050 0    60   ~ 0
-LED2\nUSART2
+STRIP2\nUSART2
 $Comp
 L SP3485CN U2
@@
 Connection ~ 2700 6000
 Text Notes 6300 2850 2    60   ~ 0
-ADC1_IN12_U1
+U1_ADC1_IN12
 Text Notes 5200 2250 2    60   ~ 0
-ADC1_IN15_U2
+U2_ADC1_IN15
 Wire Wire Line
 	6600 2700 7500 2700

Commit message: Update to KiCad 5.0.1, add debug connector
Parts:
- removed J1: J, LedControl:Jumper, symbol CONN_01X02
- removed P14: TP, LedControl:Pad, symbol CONN_01X01
- added D4: D, Diode_SMD:D_1206_3216Metric, symbol Device:D
- added P14: Conn_01x03, Connector_PinHeader_2.00mm:PinHeader_1x03_P2.00mm_Vertical, symbol Connector_Generic:Conn_01x03
- C1, C2, C3, C4: footprint Capacitors_SMD:C_0603 -> Capacitor_SMD:C_0603_1608Metric; symbol C -> Device:C
- C5: footprint Capacitors_SMD:C_1206 -> Capacitor_SMD:C_1206_3216Metric; symbol C -> Device:C
- D1: footprint LEDs:LED_0805 -> LED_SMD:LED_0805_2012Metric; symbol LED -> Device:LED
- J2: value J -> Jumper; symbol CONN_01X03 -> Connector_Generic:Conn_01x03
- J3: value CONN_01X02 -> Jumper; symbol CONN_01X02 -> Connector_Generic:Conn_01x02
- P1: symbol USB_OTG -> Connector:USB_OTG
- P10, P13, P2, P3, P32, P33, P4, P6, P7, P9: symbol CONN_01X01 -> Connector_Generic:Conn_01x01
- P11, P16, P17, P5: symbol CONN_01X02 -> Connector_Generic:Conn_01x02
- P12: symbol CONN_01X24 -> Connector_Generic:Conn_01x24
- P15: value CONN_01X01 -> TP; symbol CONN_01X01 -> Connector_Generic:Conn_01x01
- P18, P19: footprint Pin_Headers:Pin_Header_Straight_1x03 -> Connector_PinHeader_2.54mm:PinHeader_1x03_P2.54mm_Vertical; symbol CONN_01X03 -> Connector_Generic:Conn_01x03
- P8: symbol Micro_SD -> LedControl:Micro_SD_Card
- R1, R11, R3, R7: footprint Resistors_SMD:R_0603 -> Resistor_SMD:R_0603_1608Metric; symbol R -> Device:R
- R10, R2, R4, R6, R8, R9: footprint Resistors_SMD:R_1206 -> Resistor_SMD:R_1206_3216Metric; symbol R -> Device:R
- SW1, SW2: symbol ROTARY_ENCODER_SWITCH -> Device:Rotary_Encoder_Switch
- U1: footprint Housings_DFN_QFN:QFN-48-1EP_7x7mm_Pitch0.5mm -> Package_DFN_QFN:QFN-48-1EP_7x7mm_P0.5mm_EP5.6x5.6mm; symbol STM32L433CCUx -> MCU_ST_STM32L4:STM32L433CCUx
- U2, U3, U4: footprint Housings_SOIC:SOIC-8_3.9x4.9mm_Pitch1.27mm -> Package_SO:SOIC-8_3.9x4.9mm_P1.27mm; symbol SP3485CN -> Interface_UART:SP3485CN
- X1: symbol IQXO/7X -> Oscillator:IQXO-70
Connections:
- net labels added: DEBUG_LED, DISP_D_C#, DISP_MOSI, DISP_NSS, DISP_RES#, DISP_SCK, ENC1_CH1, ENC1_CH2, ENC1_SW, ENC2_CH1, ENC2_CH2, ENC2_SW, RS485_DE, RS485_RX, RS485_TX, SD_DET, SD_MISO, SD_MOSI, SD_NSS, SD_SCK, STRIP1_TTY_TX, STRIP2_DE, STRIP2_RX, STRIP2_TX, SWDCLK, SWDIO, TTY_RX, U1, U2, USB_DM, USB_DP
- wire segments 211 -> 174
Other:
- note added: "DEBUG_PORT"
- note added: "GND/PWR"
- note added: "TTY"
- note removed: "DEBUG_LED"
- note removed: "DISP_D/C#"
- note removed: "DISP_RES#"
- note removed: "ENC1_SW"
- note removed: "ENC1_TIM1_CH1"
- note removed: "ENC1_TIM1_CH2"
- note removed: "ENC2_SW"
- note removed: "ENC2_TIM2_CH1"
- note removed: "ENC2_TIM2_CH2"
- note removed: "RCC_OSC_IN"
- note removed: "RCC_OSC_OUT"
- note removed: "RS485\nGND/PWR"
- note removed: "RS485_USART3_DE"
- note removed: "RS485_USART3_RX"
- note removed: "RS485_USART3_TX"
- note removed: "SD_Cd"
- note removed: "SD_SPI1_MISO"
- note removed: "SD_SPI1_MOSI"
- note removed: "SD_SPI1_SCK"
- note removed: "SPI1_SD_NSS"
- note removed: "SPI2_DISP_MOSI"
- note removed: "SPI2_DISP_NSS"
- note removed: "SPI2_DISP_SCK"
- note removed: "STRIP1_USART1_TX"
- note removed: "STRIP2_DE"
- note removed: "STRIP2_USART2_RX"
- note removed: "STRIP2_USART2_TX"
- note removed: "U1_ADC1_IN12"
- note removed: "U2_ADC1_IN15"
- note removed: "USART1"
- note removed: "USART1_RX"
- note removed: "USB_DM"
- note removed: "USB_DP"
- moved on the sheet: U1
