File: Hardware2/Board/LedControl.sch (KiCad schematic (older format))
At the start: 75 parts, among them J2 Jumper, J3 Jumper, J4 Jumper, J5 Jumper, P1 USB_OTG, P10 Micro_SD, P11 Header, P12 DISPLAY, P13 TP, P14 TMM-103-03-G-S, P15 TP, P16 TP, P17 2059-302, P18 CONN_01X03, P19 TP, P2 2059-302, P3 2059-302, P32 TP, P33 TP, P34 TP, P36 TP, P38 TP, P39 TP, P4 2059-302, P40 TP, P41 TP, P42 TP, P43 TP, P44 TP, P5 2059-302, P6 2059-302, P7 2059-302, P8 2059-302, P9 2059-302, Q1 DMG1012UW, Q2 DMG1012UW, SW1 PEC12R-4215F-S0024, SW2 PEC12R-4215F-S0024, U1 STM32L433CCUx, U10 SP485CN, U2 SN65HVD230, U3 SP485CN, U4 SP485CN, X1 IQXO/7X

Commit message: USB and SD card at center
Parts:
- P11: footprint Connector_PinHeader_2.54mm:PinHeader_1x04_P2.54mm_Vertical -> Connector_PinHeader_2.54mm:PinHeader_1x05_P2.54mm_Vertical; symbol Connector_Generic:Conn_01x04 -> Connector_Generic:Conn_01x05
Connections:
- net +3V3: now also P11.4 (Pin_4), SW1.S1; no longer SW1.S2
- net ENC1_SW: now also SW1.S2; no longer SW1.S1
- net NRST: now also P11.5 (Pin_5); no longer P11.4 (Pin_4)
- net SWCLK: now also P11.2 (Pin_2); no longer P11.3 (Pin_3)
- net SWDIO: now also P11.3 (Pin_3); no longer P11.2 (Pin_2)
Changed lines of the file:
@@
 Text GLabel 6900 5400 0    50   Input ~ 0
 ENC2_SW
-Text GLabel 4900 5200 0    50   Input ~ 0
+Text GLabel 5100 5400 0    50   Input ~ 0
 ENC1_SW
 Text GLabel 4000 1700 0    50   Input ~ 0
@@
 Wire Wire Line
 	2100 6000 2600 6000
-Wire Wire Line
-	5100 5400 5000 5400
-Wire Wire Line
-	5000 4900 5000 5400
 $Comp
 L Interface_UART:SP3485CN U10
@@
 Wire Wire Line
 	4100 1700 4800 1700
-Wire Wire Line
-	4900 5200 5100 5200
 Connection ~ 4100 1700
 Wire Wire Line
@@
 NRST
 $Comp
-L Connector_Generic:Conn_01x04 P11
+L Connector_Generic:Conn_01x05 P11
 U 1 1 5CEA51D8
-P 3700 7500
-F 0 "P11" H 3780 7542 50  0000 L CNN
-F 1 "Header" H 3780 7451 50  0000 L CNN
-F 2 "Connector_PinHeader_2.54mm:PinHeader_1x04_P2.54mm_Vertical" H 3700 7500 50  0001 C CNN
-F 3 "~" H 3700 7500 50  0001 C CNN
-	1    3700 7500
+P 3700 7400
+F 0 "P11" H 3780 7442 50  0000 L CNN
+F 1 "Header" H 3780 7351 50  0000 L CNN
+F 2 "Connector_PinHeader_2.54mm:PinHeader_1x05_P2.54mm_Vertical" H 3700 7400 50  0001 C CNN
+F 3 "~" H 3700 7400 50  0001 C CNN
+	1    3700 7400
 	1    0    0    1
 $EndComp
@@
 	1    0    0    -1
 $EndComp
+Text GLabel 3500 7400 0    50   Input ~ 0
+SWDIO
 Text GLabel 3500 7500 0    50   Input ~ 0
-SWDIO
-Text GLabel 3500 7400 0    50   Input ~ 0
 SWCLK
-Text GLabel 3500 7300 0    50   Input ~ 0
+Text GLabel 3500 7200 0    50   Input ~ 0
 NRST
 $Comp
@@
 	7400 3500 7700 3500
 $Comp
-L power:+5V #PWR?
+L power:+5V #PWR0128
 U 1 1 5D000939
 P 7400 3200
-F 0 "#PWR?" H 7400 3050 50  0001 C CNN
+F 0 "#PWR0128" H 7400 3050 50  0001 C CNN
 F 1 "+5V" H 7400 3340 50  0000 C CNN
 F 2 "" H 7400 3200 50  0000 C CNN
@@
 $EndComp
 $Comp
-L power:+5V #PWR?
+L power:+5V #PWR0129
 U 1 1 5D0009DA
 P 7400 2300
-F 0 "#PWR?" H 7400 2150 50  0001 C CNN
+F 0 "#PWR0129" H 7400 2150 50  0001 C CNN
 F 1 "+5V" H 7400 2440 50  0000 C CNN
 F 2 "" H 7400 2300 50  0000 C CNN
@@
 	1    0    0    -1
 $EndComp
+Wire Wire Line
+	5100 5200 5000 5200
+Wire Wire Line
+	5000 5200 5000 4900
+$Comp
+L power:+3V3 #PWR?
+U 1 1 5D015D88
+P 3200 7200
+F 0 "#PWR?" H 3200 7050 50  0001 C CNN
+F 1 "+3.3V" H 3200 7340 50  0000 C CNN
+F 2 "" H 3200 7200 50  0000 C CNN
+F 3 "" H 3200 7200 50  0000 C CNN
+	1    3200 7200
+	1    0    0    -1
+$EndComp
+Wire Wire Line
+	3500 7300 3200 7300
+Wire Wire Line
+	3200 7300 3200 7200
 $EndSCHEMATC

Commit message: add rfid and speaker
Parts:
- removed P16, P19, P34, P36, P39, P41, P42, P43: TP, LedControl:Pad, symbol Connector_Generic:Conn_01x01
- added C13, C14, C20, C21: 100n, Capacitor_SMD:C_0603_1608Metric, symbol Device:C
- added C18, C19: 100p, Capacitor_SMD:C_0603_1608Metric, symbol Device:C
- added D7: SD1206S020S1R0, Diode_SMD:D_1206_3216Metric, symbol Device:D
- added J8: Jumper, LedControl:Jumper, symbol Connector_Generic:Conn_01x02
- added P16: Header, Connector_PinHeader_2.54mm:PinHeader_1x05_P2.54mm_Vertical, symbol Connector_Generic:Conn_01x05
- added P37: Header, Connector_PinHeader_2.54mm:PinHeader_1x08_P2.54mm_Vertical, symbol Connector_Generic:Conn_01x08
- added P45, P46: Header, Connector_PinHeader_2.54mm:PinHeader_1x02_P2.54mm_Vertical, symbol Connector_Generic:Conn_01x02
- added R30, R31, R32, R33: 150k, Resistor_SMD:R_0603_1608Metric, symbol Device:R
- added U11, U12: TPA2005, Package_SO:MSOP-8-1EP_3x3mm_P0.65mm_EP1.68x1.88mm, symbol LedControl:TPA2005
- C16, C17: value 100n -> 100p
- P1: value USB_OTG -> Micro_USB
- SW1, SW2: symbol Device:Rotary_Encoder_Switch -> LedControl:Rotary_Encoder_Switch
Connections:
- net U2 is gone; now on net DISP_D_C#: U1.18 (PB0)
- net +3V3: now also SW1.2 (C), SW1.4 (S1), SW2.2 (C), SW2.4 (S1), P37.8 (Pin_8); no longer SW1.C, SW1.S1, SW2.C, SW2.S1
- net +5V: now also C20.1, C21.1, J8.2 (Pin_2), P16.5 (Pin_5), U11.6 (VDD), U12.6 (VDD); no longer C16.1, C17.1
- net DISP_D_C#: no longer U1.31 (PA10)
- net DISP_NSS: now also U1.20 (PB2); no longer U1.25 (PB12)
- net ENC1_CH1: now also SW1.1 (A); no longer SW1.A
- net ENC1_CH2: now also SW1.3 (B); no longer SW1.B
- net ENC1_SW: now also SW1.5 (S2); no longer SW1.S2
- net ENC2_CH1: now also SW2.1 (A); no longer SW2.A
- net ENC2_CH2: now also SW2.3 (B); no longer SW2.B
- net ENC2_SW: now also SW2.5 (S2); no longer SW2.S2
- net GND: now also C17.2, SW1.6 (SH), SW2.6 (SH), C13.2, C14.2, C19.2, C20.2, C21.2, P16.1 (Pin_1), P37.6 (Pin_6), U11.7 (GND), U11.9 (Pad), U12.7 (GND), U12.9 (Pad)
- net RS485_RX: no longer C17.2, R28.1
- net RS485_TX: no longer C16.2, R26.1
- net SD_DET: now also U1.3 (PC14); no longer U1.27 (PB14)
- net SD_MISO: now also U1.27 (PB14); no longer U1.16 (PA6)
- net SD_NSS: now also U1.25 (PB12); no longer U1.38 (PA15)
- net STRIP1_TTY_TX: now also P16.2 (Pin_2)
- net at D1.2 (A), R22.2: now also P16.4 (Pin_4)
- net OUT2: now reaches P13.1 (Pin_1), Q2.1 (G), U1.13 (PA3)
- net OUT2: now also D7.2 (A)
- net RFID_SCK: now reaches U1.39 (PB3)
- net RFID_SCK: now also P37.2 (Pin_2)
- net RFID_MISO: now reaches U1.40 (PB4)
- net RFID_MISO: now also P37.4 (Pin_4)
- net RFID_IRQ: now reaches U1.2 (PC13)
- net RFID_IRQ: now also P37.5 (Pin_5)
- net SHUTDOWN: now reaches U1.6 (PH1)
- net SHUTDOWN: now also U11.1 (~SHUTDOWN), U12.1 (~SHUTDOWN)
- net at D4.2 (A), P1.1 (VBUS): now also J8.1 (Pin_1)
- net DEBUG_LED renamed AUDIO1
- net AUDIO1: now also C16.2; no longer R22.1
- net DISP_MOSI renamed DISP_SD_MOSI
- net DISP_SD_MOSI: now also P10.3 (CMD)
- net DISP_RES# renamed DISP_RFID_RES#
- net DISP_RFID_RES#: now also U1.31 (PA10), P37.7 (Pin_7); no longer U1.20 (PB2)
- net DISP_SCK renamed DISP_SD_SCK
- net DISP_SD_SCK: now also P10.5 (CLK)
- net SD_MOSI renamed RFID_MOSI
- net RFID_MOSI: now also P37.3 (Pin_3); no longer P10.3 (CMD)
- net SD_SCK renamed AUDIO2
- net AUDIO2: now also C18.2; no longer P10.5 (CLK)
- net STRIP2_TX renamed STRIP2_TX_OUT1
- net TTY_RX renamed LED_TTY_RX
- net LED_TTY_RX: now also R22.1, P16.3 (Pin_3)
- net U1 renamed IN2
- net IN2: now also R28.1, C14.1
- new net: C16.1, R30.2
- new net: R30.1, U11.3 (IN+)
- new net: R31.1, U11.4 (IN-)
- new net: C17.1, R31.2
- new net: P45.2 (Pin_2), U11.5 (VO+)
- new net: P45.1 (Pin_1), U11.8 (VO-)
- new net: R32.1, U12.3 (IN+)
- new net: R33.1, U12.4 (IN-)
- new net: P46.2 (Pin_2), U12.5 (VO+)
- new net: P46.1 (Pin_1), U12.8 (VO-)
- new net: C18.1, R32.2
- new net: C19.1, R33.2
- new net IN1: C13.1, R26.1, U1.16 (PA6)
- new net Power/EN: D7.1 (K)
- new net RFID_NSS: P37.1 (Pin_1), U1.38 (PA15)
Other:
- note added: "AUDIO"
- note added: "Alternative to RS485 and U1/U2"
- note added: "DEBUG PORT"
- note added: "ENCODER 1/2\nTIM1/2"
- note added: "RFID\nMFRC522\nSPI3"
- note removed: "Alternative to RS485"
- note removed: "DEBUG_PORT"
- note removed: "ENCODER 1\nTIM1"
- note removed: "ENCODER 2\nTIM2"
- moved on the sheet: C1, D1, D5, D6, P11, P13, P14, P33, P44, Q1, Q2, R1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
